File: hardware/pcbs/audio_board/audio_board.kicad_sch (KiCad schematic)
At the start: 23 parts, among them J1 Conn_02x07_Odd_Even, J2 MTA100_08, J3 NC3MAH, J4 AudioJack3, J5 NC3MAH, U1 Teensy 4.1

Commit message: minor changes
Other:
- title: FOSDEM audio V2 -> FOSDEM audio rev G
Changed lines of the file:
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@@
 	(paper "A4")
 	(title_block
-		(title "FOSDEM audio V2")
+		(title "FOSDEM audio rev G")
 		(rev "1")
 		(comment 1 "3 balanced inputs, 2 balanced outputs, 1 mono line-in")
