File: hardware/pcbs/audio_board/clock_fanout.kicad_sch (KiCad schematic)
At the start: 14 parts, among them U7 LMK1C1103A, U8 LMK1C1103A

Commit message: audioboard: BOM fixes
Parts:
- FB1: MPN BLM21PG102SN1D -> BLM21AG102SN1D
Changed lines of the file:
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@@
 			)
 		)
-		(property "MPN" "BLM21PG102SN1D"
+		(property "MPN" "BLM21AG102SN1D"
 			(at 101.6 82.55 90)
 			(hide yes)
