File: hardware/pcbs/audio_board/input_mono.kicad_sch (KiCad schematic)
At the start: 10 parts, among them J9 AudioJack3

Commit message: audioboard: BOM fixes
Parts:
- C60: MPN C 1nF LowESR 100V 0805 -> C 1nF Audio 100V 0805
- C61, C62: MPN C 10μF LowESR 100V P2 -> C 10μF Audio 100V P2
Changed lines of the file:
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@@
 			)
 		)
-		(property "MPN" "C 10μF LowESR 100V P2"
+		(property "MPN" "C 10μF Audio 100V P2"
 			(at 147.32 123.19 90)
 			(hide yes)
@@
 			)
 		)
-		(property "MPN" "C 1nF LowESR 100V 0805"
+		(property "MPN" "C 1nF Audio 100V 0805"
 			(at 128.27 109.22 0)
 			(hide yes)
@@
 			)
 		)
-		(property "MPN" "C 10μF LowESR 100V P2"
+		(property "MPN" "C 10μF Audio 100V P2"
 			(at 147.32 95.25 90)
 			(hide yes)
