File: hardware/pcbs/audio_board/xlr_input.kicad_sch (KiCad schematic)
At the start: 24 parts, among them J6 NC3FAH1, Q2 2N7002, Q3 SI2309CDS-T1-GE3

Commit message: audioboard: BOM fixes
Parts:
- C39, C40: MPN C 1nF LowESR 100V 0805 -> C 1nF Audio 100V 0805
- C42: MPN C 2.2nF LowESR 100V 0805 -> C 2.2nF Audio 100V 0805
- C43, C44: MPN C 10μF LowESR 100V P2 -> C 10μF Audio 100V P2
Changed lines of the file:
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@@
 			(justify left bottom)
 		)
-		(property "Net Class" "Phantom"
+		(property "Netclass" "Phantom"
 			(at 85.7885 45.72 0)
 			(show_name no)
@@
 			(justify left bottom)
 		)
-		(property "Net Class" "Phantom"
+		(property "Netclass" "Phantom"
 			(at 69.85 58.9915 90)
 			(show_name no)
@@
 			(justify left bottom)
 		)
-		(property "Net Class" "Phantom"
+		(property "Netclass" "Phantom"
 			(at 128.9685 102.87 0)
 			(show_name no)
@@
 			(justify right bottom)
 		)
-		(property "Net Class" "Phantom"
+		(property "Netclass" "Phantom"
 			(at 68.0085 125.73 0)
 			(show_name no)
@@
 			(justify left bottom)
 		)
-		(property "Net Class" "Phantom"
+		(property "Netclass" "Phantom"
 			(at 88.392 65.786 0)
 			(show_name no)
@@
 			(justify left bottom)
 		)
-		(property "Net Class" "Phantom"
+		(property "Netclass" "Phantom"
 			(at 88.392 55.626 0)
 			(show_name no)
@@
 			(justify left bottom)
 		)
-		(property "Net Class" "Phantom"
+		(property "Netclass" "Phantom"
 			(at 68.0085 102.87 0)
 			(show_name no)
@@
 			(justify left bottom)
 		)
-		(property "Net Class" "Phantom"
+		(property "Netclass" "Phantom"
 			(at 85.7885 31.75 0)
 			(show_name no)
@@
 			(justify left bottom)
 		)
-		(property "Net Class" "Phantom"
+		(property "Netclass" "Phantom"
 			(at 105.918 100.584 0)
 			(show_name no)
@@
 			(justify right bottom)
 		)
-		(property "Net Class" "Phantom"
+		(property "Netclass" "Phantom"
 			(at 95.9485 125.73 0)
 			(show_name no)
@@
 			(justify right bottom)
 		)
-		(property "Net Class" "Phantom"
+		(property "Netclass" "Phantom"
 			(at 128.9685 125.73 0)
 			(show_name no)
@@
 			)
 		)
-		(property "MPN" "C 10μF LowESR 100V P2"
+		(property "MPN" "C 10μF Audio 100V P2"
 			(at 161.29 100.33 90)
 			(hide yes)
@@
 			)
 		)
-		(property "MPN" "C 1nF LowESR 100V 0805"
+		(property "MPN" "C 1nF Audio 100V 0805"
 			(at 80.01 118.11 0)
 			(hide yes)
@@
 			)
 		)
-		(property "MPN" "C 2.2nF LowESR 100V 0805"
+		(property "MPN" "C 2.2nF Audio 100V 0805"
 			(at 154.94 114.3 0)
 			(hide yes)
@@
 			)
 		)
-		(property "MPN" "C 10μF LowESR 100V P2"
+		(property "MPN" "C 10μF Audio 100V P2"
 			(at 161.29 128.27 90)
 			(hide yes)
@@
 			)
 		)
-		(property "MPN" "C 1nF LowESR 100V 0805"
+		(property "MPN" "C 1nF Audio 100V 0805"
 			(at 80.01 110.49 0)
 			(hide yes)
