File: hardware/pcbs/audio_board/audio_board.kicad_pcb (KiCad board)
At the start: 4 copper layers, 152 x 61.5 mm, 180 parts, among them J1 Conn_02x07_Odd_Even, J2 MTA100_08, J3 NC3MAH, J4 AudioJack3, J5 NC3MAH, J6 NC3FAH1, J7 NC3FAH1, J8 NC3FAH1, J9 AudioJack3, Q1 S8050, Q2 2N7002, Q3 SI2309CDS-T1-GE3, Q4 2N7002, Q5 SI2309CDS-T1-GE3, Q6 2N7002, Q7 SI2309CDS-T1-GE3, U1 Teensy 4.1, U2 LP5907MFX-3.3, U3 LM5158, U4 TAD5242, U5 TAD5242, U6 TAA3040, U7 LMK1C1103A, U8 LMK1C1103A

Commit message: audio_board: fix backside revision
Other:
- board text removed: "FOSDEM Audio Interface rev. F"
Changed lines of the file:
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@@
 		)
 	)
-	(gr_text "FOSDEM Audio Interface rev. F"
+	(gr_text "FOSDEM Audio Interface rev. G"
 		(at 220 100 90)
 		(layer "B.SilkS")

Commit message: audio_board: update silkscreen for final revH
Routing:
- net GND: vias 434 -> 433
Other:
- board text added: "FOSDEM Audio Interface rev. H"
- board text added: "HEADPHONE"
- board text added: "IN PC (MONO)"
- board text added: "IN1"
- board text added: "IN2"
- board text added: "IN3"
- board text added: "OUT1"
- board text added: "OUT2"
- board text removed: "FOSDEM Audio Interface rev. G"
Changed lines of the file:
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@@
 		(tags "resistor")
 		(property "Reference" "R30"
-			(at -2.070586 -0.007446 180)
+			(at 1.943523 -0.122236 180)
 			(layer "F.SilkS")
 			(effects
@@
 		(tags "capacitor")
 		(property "Reference" "C60"
-			(at 1.956711 -0.107126 180)
+			(at -0.0375 -1.265 270)
 			(layer "F.SilkS")
 			(effects
@@
 		(tags "resistor")
 		(property "Reference" "R69"
-			(at -1.96 0.04 270)
+			(at 1.870303 -0.001804 270)
 			(layer "F.SilkS")
 			(effects
@@
 		(tags "resistor")
 		(property "Reference" "R70"
-			(at -1.96 0.04 270)
+			(at 1.843209 -0.000641 270)
 			(layer "F.SilkS")
 			(effects
@@
 		(tags "inductor")
 		(property "Reference" "L4"
-			(at -2.032142 -0.000292 180)
+			(at 1.925 -0.000292 180)
 			(layer "F.SilkS")
 			(effects
@@
 		(tags "TRS audio jack stereo horizontal circular")
 		(property "Reference" "J9"
-			(at -5.019633 0.610741 240)
+			(at -2.580144 13.63606 330)
 			(layer "F.SilkS")
 			(effects
@@
 		(layer "User.6")
 	)
-	(gr_text "FOSDEM Audio Interface rev. G"
+	(gr_text "FOSDEM Audio Interface rev. H"
 		(at 220 123.5 90)
 		(layer "F.SilkS")
@@
 		)
 	)
-	(gr_text "FOSDEM Audio Interface rev. G"
+	(gr_text "OUT1"
+		(at 88.75 130.25 0)
+		(layer "F.SilkS")
+		(effects
+			(font
+				(size 1 1)
+				(thickness 0.15)
+			)
+			(justify bottom)
+		)
+	)
+	(gr_text "OUT2"
+		(at 115.75 130.25 0)
+		(layer "F.SilkS")
+		(effects
+			(font
+				(size 1 1)
+				(thickness 0.15)
+			)
+			(justify bottom)
+		)
+	)
+	(gr_text "IN1"
+		(at 145.5 130.1 0)
+		(layer "F.SilkS")
+		(effects
+			(font
+				(size 1 1)
+				(thickness 0.15)
+			)
+			(justify bottom)
+		)
+	)
+	(gr_text "IN2"
+		(at 172.6 130 0)
+		(layer "F.SilkS")
+		(effects
+			(font
+				(size 1 1)
+				(thickness 0.15)
+			)
+			(justify bottom)
+		)
+	)
+	(gr_text "IN3"
+		(at 199.5 130.1 0)
+		(layer "F.SilkS")
+		(effects
+			(font
+				(size 1 1)
+				(thickness 0.15)
+			)
+			(justify bottom)
+		)
+	)
+	(gr_text "HEADPHONE"
+		(at 215.1 134.3 0)
+		(layer "F.SilkS")
+		(effects
+			(font
+				(size 1 1)
+				(thickness 0.15)
+			)
+			(justify bottom)
+		)
+	)
+	(gr_text "IN PC (MONO)"
+		(at 197.792101 97.75293 60)
+		(layer "F.SilkS")
+		(effects
+			(font
+				(size 1 1)
+				(thickness 0.15)
+			)
+			(justify bottom)
+		)
+	)
+	(gr_text "FOSDEM Audio Interface rev. H"
 		(at 220 100 90)
 		(layer "B.SilkS")
@@
 		(net "GND")
 	)
-	(via
-		(at 198 96)
-		(size 0.6)
-		(drill 0.3)
-		(layers "F.Cu" "B.Cu")
-		(capping no)
-		(covering
-			(front no)
-			(back no)
-		)
-		(plugging
-			(front no)
-			(back no)
-		)
-		(filling no)
-		(net "GND")
-	)
